File: 1inch-photodetector.kicad_sch (KiCad schematic)
At the start: 23 parts, among them J1 Conn_01x03, J2 Conn_Coaxial, U1 ADA4898-2, U2 LT3032IDE-12

Commit message: Fixed white spaces
Parts:
- J1: PN 53398-0371 -> 53398-0371
- U2: Alternative Analog Devices LT3032EDE-12#PBF -> Analog Devices LT3032EDE-12#PBF; PN LT3032IDE-12#PBF -> LT3032IDE-12#PBF
Changed lines of the file:
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@@
 			)
 		)
-		(property "PN" " 53398-0371"
+		(property "PN" "53398-0371"
 			(at 29.21 144.78 0)
 			(effects
@@
 			)
 		)
-		(property "PN" "LT3032IDE-12#PBF "
+		(property "PN" "LT3032IDE-12#PBF"
 			(at 80.01 156.21 0)
 			(effects
@@
 			)
 		)
-		(property "Alternative" "Analog Devices LT3032EDE-12#PBF "
+		(property "Alternative" "Analog Devices LT3032EDE-12#PBF"
 			(at 80.01 156.21 0)
 			(effects
@@
 			)
 		)
-		(property "PN" "LT3032IDE-12#PBF "
+		(property "PN" "LT3032IDE-12#PBF"
 			(at 80.01 134.62 0)
 			(effects
@@
 			)
 		)
-		(property "Alternative" "Analog Devices LT3032EDE-12#PBF "
+		(property "Alternative" "Analog Devices LT3032EDE-12#PBF"
 			(at 80.01 134.62 0)
 			(effects
