File: 1inch-photodetector.kicad_pcb (KiCad board)
At the start: 4 copper layers, 25.4 x 25.4 mm, 23 parts, among them J1 Conn_01x03, J2 Conn_Coaxial, U1 ADA4898-2, U2 LT3032IDE-12

Commit message: Fix stackup. An incorrect stackup was given. Changed to PCBWay/JLCPCB standard. (#16)
- Bump version to 1.1.1
Other:
- board text added: "0,203 mm"
- board text added: "1,03 mm"
- board text added: "4,6"
- board text added: "4,74"
- board text added: "Dielectric 1"
- board text added: "Dielectric 2"
- board text added: "Dielectric 3"
- board text added: "Liquid Ink"
- board text removed: "0,1 mm"
- board text removed: "1,24 mm"
- board text removed: "4,5"
- board text removed: "Dielectric"
